Commit message: Cleaning up launch files.

File: packages/my_gazebo_worlds/worlds/empty.world.xacro (robot description, xacro)
@@ -19,4 +19,38 @@
   xmlns:physics="http://playerstage.sourceforge.net/gazebo/xmlschema/#physics"
   >
+  <!--=========================-->
+  <!-- BEGIN XACRO DEFINITIONS -->
+  <!--=========================-->
+  <!-- Ground plane size in metres (both x and y) -->
+  <xacro:property name="ground_plane_size"  value="100" />
+  <!-- Range and height for each light -->
+  <xacro:property name="light_range"        value="${ground_plane_size/4}" />
+  <xacro:property name="light_height"       value="10" />
+  <!-- Macro to create one point light at given position -->
+  <xacro:macro name="light_macro" params="n x y z">
+    <model:renderable name="light_${n}">
+      <xyz>${x} ${y} ${z}</xyz>
+      <rpy>0.0 0.0 0</rpy>
+      <enableGravity>false</enableGravity>
+      <light>
+        <type>point</type>
+        <diffuseColor>0.8 0.8 0.8</diffuseColor>
+        <specularColor>.1 .1 .1</specularColor>
+        <attenuation>0.2 0.1 0</attenuation>
+        <range>${light_range}</range>
+      </light>
+    </model:renderable>
+  </xacro:macro>
+  <!-- Macro to create point lights distributed around the world -->
+  <xacro:macro name="lights_macro">
+    <xacro:light_macro n="1" x="0"                y="0"               z="${light_height}" />
+    <xacro:light_macro n="2" x="${light_range}"   y="${light_range}"  z="${light_height}" />
+    <xacro:light_macro n="3" x="${light_range}"   y="-${light_range}" z="${light_height}" />
+    <xacro:light_macro n="4" x="-${light_range}"  y="${light_range}"  z="${light_height}" />
+    <xacro:light_macro n="5" x="-${light_range}"  y="-${light_range}" z="${light_height}" />
+  </xacro:macro>
+  <!--=========================-->
+  <!-- END XACRO DEFINITIONS   -->
+  <!--=========================-->
   <thread>4</thread>
   <verbosity>5</verbosity>
@@ -70,5 +104,5 @@
         <kd>1.0</kd>
         <normal>0 0 1</normal>
-        <size>100 100</size>
+        <size>${ground_plane_size} ${ground_plane_size}</size>
         <segments>10 10</segments>
         <uvTile>200 400</uvTile>
@@ -77,22 +111,4 @@
     </body:plane>
   </model:physical>
-  <xacro:macro name="light_macro" params="n x y z">
-    <model:renderable name="light_${n}">
-      <xyz>${x} ${y} ${z}</xyz>
-      <rpy>0.0 0.0 0</rpy>
-      <enableGravity>false</enableGravity>
-      <light>
-        <type>point</type>
-        <diffuseColor>0.8 0.8 0.8</diffuseColor>
-        <specularColor>.1 .1 .1</specularColor>
-        <attenuation>0.2 0.1 0</attenuation>
-        <range>25</range>
-      </light>
-    </model:renderable>
-  </xacro:macro>
-  <xacro:light_macro n="1" x="0"   y="0"   z="10" />
-  <xacro:light_macro n="2" x="20"  y="20"  z="10" />
-  <xacro:light_macro n="3" x="20"  y="-20" z="10" />
-  <xacro:light_macro n="4" x="-20" y="20"  z="10" />
-  <xacro:light_macro n="5" x="-20" y="-20" z="10" />
+  <xacro:lights_macro/>
 </gazebo:world>

Commit message: Updating xacro handling and models.

File: packages/my_gazebo_worlds/worlds/empty.world.xacro (robot description, xacro)
@@ -1,5 +1,4 @@
 <?xml version="1.0"?>
 <gazebo:world
-  xmlns:xacro="http://www.ros.org/wiki/xacro"
   xmlns:xi="http://www.w3.org/2001/XInclude"
   xmlns:gazebo="http://playerstage.sourceforge.net/gazebo/xmlschema/#gz"
@@ -18,15 +17,16 @@
   xmlns:controller="http://playerstage.sourceforge.net/gazebo/xmlschema/#controller"
   xmlns:physics="http://playerstage.sourceforge.net/gazebo/xmlschema/#physics"
+  xmlns:xacro="http://www.ros.org/wiki/xacro"
   >
-  <!--=========================-->
-  <!-- BEGIN XACRO DEFINITIONS -->
-  <!--=========================-->
+  <!-- ============================ -->
+  <!-- BEGIN XACRO DEFINITIONS      -->
+  <!-- ============================ -->
   <!-- Ground plane size in metres (both x and y) -->
-  <xacro:property name="ground_plane_size"  value="100" />
+  <xacro:property name="GROUND_PLANE_SIZE"  value="100" />
   <!-- Range and height for each light -->
-  <xacro:property name="light_range"        value="${ground_plane_size/4}" />
-  <xacro:property name="light_height"       value="10" />
+  <xacro:property name="LIGHT_RANGE"        value="${GROUND_PLANE_SIZE/4}" />
+  <xacro:property name="LIGHT_HEIGHT"       value="10" />
   <!-- Macro to create one point light at given position -->
-  <xacro:macro name="light_macro" params="n x y z">
+  <xacro:macro name="LIGHT_MACRO" params="n x y z">
     <model:renderable name="light_${n}">
       <xyz>${x} ${y} ${z}</xyz>
@@ -38,19 +38,19 @@
         <specularColor>.1 .1 .1</specularColor>
         <attenuation>0.2 0.1 0</attenuation>
-        <range>${light_range}</range>
+        <range>${LIGHT_RANGE}</range>
       </light>
     </model:renderable>
   </xacro:macro>
   <!-- Macro to create point lights distributed around the world -->
-  <xacro:macro name="lights_macro">
-    <xacro:light_macro n="1" x="0"                y="0"               z="${light_height}" />
-    <xacro:light_macro n="2" x="${light_range}"   y="${light_range}"  z="${light_height}" />
-    <xacro:light_macro n="3" x="${light_range}"   y="-${light_range}" z="${light_height}" />
-    <xacro:light_macro n="4" x="-${light_range}"  y="${light_range}"  z="${light_height}" />
-    <xacro:light_macro n="5" x="-${light_range}"  y="-${light_range}" z="${light_height}" />
+  <xacro:macro name="LIGHTS_MACRO">
+    <xacro:LIGHT_MACRO n="1" x="0"                y="0"               z="${LIGHT_HEIGHT}" />
+    <xacro:LIGHT_MACRO n="2" x="${LIGHT_RANGE}"   y="${LIGHT_RANGE}"  z="${LIGHT_HEIGHT}" />
+    <xacro:LIGHT_MACRO n="3" x="${LIGHT_RANGE}"   y="-${LIGHT_RANGE}" z="${LIGHT_HEIGHT}" />
+    <xacro:LIGHT_MACRO n="4" x="-${LIGHT_RANGE}"  y="${LIGHT_RANGE}"  z="${LIGHT_HEIGHT}" />
+    <xacro:LIGHT_MACRO n="5" x="-${LIGHT_RANGE}"  y="-${LIGHT_RANGE}" z="${LIGHT_HEIGHT}" />
   </xacro:macro>
-  <!--=========================-->
-  <!-- END XACRO DEFINITIONS   -->
-  <!--=========================-->
+  <!-- ============================ -->
+  <!-- END XACRO DEFINITIONS        -->
+  <!-- ============================ -->
   <thread>4</thread>
   <verbosity>5</verbosity>
@@ -104,5 +104,5 @@
         <kd>1.0</kd>
         <normal>0 0 1</normal>
-        <size>${ground_plane_size} ${ground_plane_size}</size>
+        <size>${GROUND_PLANE_SIZE} ${GROUND_PLANE_SIZE}</size>
         <segments>10 10</segments>
         <uvTile>200 400</uvTile>
@@ -111,4 +111,4 @@
     </body:plane>
   </model:physical>
-  <xacro:lights_macro/>
+  <xacro:LIGHTS_MACRO/>
 </gazebo:world>
