Commit message: Updating launch, model, and world files.

File: packages/my_gazebo_worlds/models/pioneer3dx.urdf (robot description, URDF)
Before this commit: robot pioneer3dx, 11 links, 10 joints
Links:
- removed link p3dx_left_hubcap
- removed link p3dx_left_wheel
- removed link p3dx_right_hubcap
- removed link p3dx_right_wheel
- added link left_hubcap, mass 0.01; collision box size=0 0 0; visual mesh filename=package://p2os_urdf/meshes/p3dx_meshes/left_hubcap.stl
- added link left_wheel, mass 0.5; collision cylinder length=0.01 radius=0.09; visual mesh filename=package://p2os_urdf/meshes/p3dx_meshes/left_wheel.stl
- added link right_hubcap, mass 0.01; collision box size=0 0 0; visual mesh filename=package://p2os_urdf/meshes/p3dx_meshes/right_hubcap.stl
- added link right_wheel, mass 0.5; collision cylinder length=0.01 radius=0.09; visual mesh filename=package://p2os_urdf/meshes/p3dx_meshes/right_wheel.stl
Joints:
- joint base_left_hubcap_joint: child p3dx_left_hubcap -> left_hubcap; parent p3dx_left_wheel -> left_wheel
- joint base_left_wheel_joint: child p3dx_left_wheel -> left_wheel
- joint base_right_hubcap_joint: child p3dx_right_hubcap -> right_hubcap; parent p3dx_right_wheel -> right_wheel
- joint base_right_wheel_joint: child p3dx_right_wheel -> right_wheel

File: packages/my_gazebo_worlds/models/pioneer3dx.urdf.xacro (robot description, xacro)
@@ -9,20 +9,28 @@
   <!-- BEGIN XACRO DEFINITIONS      -->
   <!-- ============================ -->
-  <!-- PI -->
+  <!-- Define PI -->
   <xacro:property name="PI" value="3.14159" />
+  <!-- Wheel moments of inertia -->
+  <xacro:property name="IXX" value="0.012411765597" />
+  <xacro:property name="IYY" value="0.015218160428" />
+  <xacro:property name="IZZ" value="0.011763977943" />
+  <xacro:property name="IXY" value="0.0"            />
+  <xacro:property name="IXZ" value="0.0"            />
+  <xacro:property name="IYZ" value="0.0"            />
   <!-- Macro to create a wheel -->
-  <xacro:macro name="P3DX_WHEEL" params="suffix parent reflect">
-    <link name="p3dx_${suffix}_wheel">
+  <xacro:macro name="WHEEL" params="name parent reflect">
+    <!-- Wheel -->
+    <link name="${name}_wheel">
       <inertial>
         <mass value="0.5"/>
         <origin xyz="0 0 0"/>
-        <inertia ixx="0.012411765597" iyy="0.015218160428" izz="0.011763977943" ixy="0" ixz="0" iyz="0" />
+        <inertia ixx="${IXX}" iyy="${IYY}" izz="${IZZ}" ixy="${IXY}" ixz="${IXZ}" iyz="${IYZ}"/>
       </inertial>
-      <visual name="base_visual">
+      <visual>
         <origin xyz="0 0 0" rpy="0 0 0"/>
-        <geometry name="pioneer_geom">
-          <mesh filename="package://p2os_urdf/meshes/p3dx_meshes/${suffix}_wheel.stl"/>
-        </geometry>
-        <material name="WheelBlack">
+        <geometry>
+          <mesh filename="package://p2os_urdf/meshes/p3dx_meshes/${name}_wheel.stl"/>
+        </geometry>
+        <material name="WheelBlack" >
           <color rgba="0.117 0.117 0.117 1"/>
         </material>
@@ -35,49 +43,5 @@
       </collision>
     </link>
-    <joint name="base_${suffix}_hubcap_joint" type="fixed">
-      <origin xyz="0 0 0" rpy="0 0 0"/>
-      <parent link="p3dx_${suffix}_wheel"/>
-      <child link="p3dx_${suffix}_hubcap"/>
-    </joint>
-    <link name="p3dx_${suffix}_hubcap">
-      <inertial>
-        <mass value="0.01"/>
-        <origin xyz="0 0 0"/>
-        <inertia ixx="0.012411765597" iyy="0.015218160428" izz="0.011763977943" ixy="0" ixz="0" iyz="0" />
-      </inertial>
-      <visual name="base_visual">
-        <origin xyz="0 0 0" rpy="0 0 0"/>
-        <geometry name="pioneer_geom">
-          <mesh filename="package://p2os_urdf/meshes/p3dx_meshes/${suffix}_hubcap.stl"/>
-        </geometry>
-        <material name="HubcapYellow">
-          <color rgba="1.0 0.811 0.151 1.0"/>
-        </material>
-      </visual>
-      <collision>
-        <origin xyz="0 0 0" rpy="0 0 0"/>
-        <geometry>
-          <box size="0 0 0"/>
-        </geometry>
-      </collision>
-    </link>
-    <transmission type="pr2_mechanism_model/SimpleTransmission" name="${parent}_${suffix}_wheel_trans">
-      <actuator name="base_${suffix}_wheel_motor" />
-      <joint name="base_${suffix}_wheel_joint" />
-      <mechanicalReduction>${reflect * 624/35 * 80/19}</mechanicalReduction>
-    </transmission>
-    <joint name="base_${suffix}_wheel_joint" type="continuous">
-      <axis xyz="0 1 0"/>
-      <anchor xyz="0 0 0"/>
-      <limit effort="100" velocity="100" />
-      <joint_properties damping="0.0" friction="0.0" />
-      <origin xyz="0 ${reflect*0.158} 0.091" rpy="0 0 0"/>
-      <parent link="base_link"/>
-      <child link="p3dx_${suffix}_wheel"/>
-    </joint>
-    <gazebo reference="p3dx_${suffix}_hubcap">
-      <material value="Gazebo/Yellow"/>
-    </gazebo>
-    <gazebo reference="p3dx_${suffix}_wheel">
+    <gazebo reference="${name}_wheel">
       <material value="Gazebo/Black"/>
       <elem key="mu1" value="0.5" />
@@ -86,9 +50,58 @@
       <elem key="kd"  value="1.0" />
     </gazebo>
+    <!-- Hubcap -->
+    <link name="${name}_hubcap">
+      <inertial>
+        <mass value="0.01"/>
+        <origin xyz="0 0 0"/>
+        <inertia ixx="${IXX}" iyy="${IYY}" izz="${IZZ}" ixy="${IXY}" ixz="${IXZ}" iyz="${IYZ}"/>
+      </inertial>
+      <visual>
+        <origin xyz="0 0 0" rpy="0 0 0"/>
+        <geometry>
+          <mesh filename="package://p2os_urdf/meshes/p3dx_meshes/${name}_hubcap.stl"/>
+        </geometry>
+        <material name="HubcapYellow" >
+          <color rgba="1.0 0.811 0.151 1.0"/>
+        </material>
+      </visual>
+      <collision>
+        <origin xyz="0 0 0" rpy="0 0 0"/>
+        <geometry>
+          <box size="0 0 0"/>
+        </geometry>
+      </collision>
+    </link>
+    <gazebo reference="${name}_hubcap">
+      <material value="Gazebo/Yellow"/>
+    </gazebo>
+    <!-- Join the wheel and hubcap -->
+    <joint name="base_${name}_hubcap_joint" type="fixed">
+      <parent link="${name}_wheel"/>
+      <child link="${name}_hubcap"/>
+      <origin xyz="0 0 0" rpy="0 0 0"/>
+    </joint>
+    <!-- Join the wheel and chassis -->
+    <joint name="base_${name}_wheel_joint" type="continuous">
+      <parent link="base_link"/>
+      <child link="${name}_wheel"/>
+      <axis xyz="0 1 0"/>
+      <anchor xyz="0 0 0"/>
+      <limit effort="100" velocity="100" />
+      <joint_properties damping="0.0" friction="0.0" />
+      <origin xyz="0 ${reflect*0.158} 0.091" rpy="0 0 0"/>
+    </joint>
+    <!--
+    <transmission name="${parent}_${name}_wheel_trans" type="pr2_mechanism_model/SimpleTransmission">
+      <actuator name="base_${name}_wheel_motor" />
+      <joint name="base_${name}_wheel_joint" />
+      <mechanicalReduction>${reflect * 624/35 * 80/19}</mechanicalReduction>
+    </transmission>
+    -->
   </xacro:macro>
   <!-- ============================ -->
   <!-- END XACRO DEFINITIONS        -->
   <!-- ============================ -->
-  <!-- Chassis -->
+  <!-- Base link -->
   <link name="base_link">
     <inertial>
@@ -116,5 +129,5 @@
     <material value="Gazebo/Red"/>
   </gazebo>
-  <!-- Top -->
+  <!-- Top plate -->
   <link name="top_plate">
     <inertial>
@@ -142,4 +155,5 @@
     <material value="Gazebo/Black"/>
   </gazebo>
+  <!-- Join the top_plate and base_link -->
   <joint name="base_top_joint" type="fixed">
     <origin xyz="-0.045 0 0.234" rpy="0 0 0"/>
@@ -154,20 +168,20 @@
       <inertia ixx="0.01" ixy="0" ixz="0"
          iyy="0.01" iyz="0" izz="0.01"/>
-      </inertial>
-  <visual name="base_visual">
-    <origin xyz="0 0 0" rpy="0 0 0"/>
-    <geometry name="pioneer_geom">
-      <mesh filename="package://p2os_urdf/meshes/p3dx_meshes/swivel.stl"/>
-    </geometry>
-    <material name="swivel">
-      <color rgba="0.5 0.5 0.5 1"/>
-    </material>
-  </visual>
-  <collision>
-    <origin xyz="0 0 0" rpy="0 0 0"/>
-    <geometry>
-      <box size="0 0 0"/>
-    </geometry>
-  </collision>
+    </inertial>
+    <visual name="base_visual">
+      <origin xyz="0 0 0" rpy="0 0 0"/>
+      <geometry name="pioneer_geom">
+        <mesh filename="package://p2os_urdf/meshes/p3dx_meshes/swivel.stl"/>
+      </geometry>
+      <material name="swivel">
+        <color rgba="0.5 0.5 0.5 1"/>
+      </material>
+    </visual>
+    <collision>
+      <origin xyz="0 0 0" rpy="0 0 0"/>
+      <geometry>
+        <box size="0 0 0"/>
+      </geometry>
+    </collision>
   </link>
   <gazebo reference="swivel">
@@ -175,4 +189,6 @@
   </gazebo>
   <joint name="base_swivel_joint" type="continuous">
+    <parent link="base_link"/>
+    <child link="swivel"/>
     <origin xyz="-0.185 0 0.055" rpy="0 0 0"/>
     <axis xyz="0 0 1"/>
@@ -180,30 +196,27 @@
     <limit effort="100" velocity="100" k_velocity="0" />
     <joint_properties damping="0.0" friction="0.0" />
-    <parent link="base_link"/>
-    <child link="swivel"/>
-  </joint>
-<!-- Center Wheel + Hubcap -->
+  </joint>
+  <!-- Center Wheel + Hubcap -->
   <link name="center_hubcap">
     <inertial>
       <mass value="0.01"/>
       <origin xyz="0 0 0"/>
-      <inertia ixx="0.012411765597" ixy="-0.000711733678" ixz="0.00050272983"
-         iyy="0.015218160428" iyz="-0.000004273467" izz="0.011763977943"/>
-      </inertial>
-  <visual name="base_visual">
-    <origin xyz="0 0 0" rpy="0 0 0"/>
-    <geometry name="pioneer_geom">
-      <mesh filename="package://p2os_urdf/meshes/p3dx_meshes/center_hubcap.stl"/>
-    </geometry>
-    <material name="swivel">
-      <color rgba="0.5 0.5 0.5 1"/>
-    </material>
-  </visual>
-  <collision>
-    <origin xyz="0 0 0" rpy="0 0 0"/>
-    <geometry>
-      <box size="0 0 0"/>
-    </geometry>
-  </collision>
+      <inertia ixx="0.012411765597" ixy="-0.000711733678" ixz="0.00050272983" iyy="0.015218160428" iyz="-0.000004273467" izz="0.011763977943"/>
+    </inertial>
+    <visual name="base_visual">
+      <origin xyz="0 0 0" rpy="0 0 0"/>
+      <geometry name="pioneer_geom">
+        <mesh filename="package://p2os_urdf/meshes/p3dx_meshes/center_hubcap.stl"/>
+      </geometry>
+      <material name="swivel">
+        <color rgba="0.5 0.5 0.5 1"/>
+      </material>
+    </visual>
+    <collision>
+      <origin xyz="0 0 0" rpy="0 0 0"/>
+      <geometry>
+        <box size="0 0 0"/>
+      </geometry>
+    </collision>
   </link>
   <gazebo reference="center_hubcap">
@@ -223,29 +236,23 @@
       <mass value="0.1"/>
       <origin xyz="0 0 0"/>
-      <inertia ixx="0.012411765597" ixy="-0.000711733678" ixz="0.00050272983"
-         iyy="0.015218160428" iyz="-0.000004273467" izz="0.011763977943"/>
-      </inertial>
-  <visual name="base_visual">
-    <origin xyz="0 0 0" rpy="0 0 0"/>
-    <geometry name="pioneer_geom">
-      <mesh filename="package://p2os_urdf/meshes/p3dx_meshes/center_wheel.stl"/>
-    </geometry>
-    <material name="WheelBlack">
-      <color rgba="0.117 0.117 0.117 1"/>
-    </material>
-  </visual>
-  <collision>
-    <origin xyz="0 0 0" rpy="${-PI/2.0} 0 0"/>
-    <geometry>
-      <!--<mesh filename="package://p2os_urdf/meshes/p3dx_meshes/center_wheel.stl"/>-->
-      <cylinder radius="0.0375" length="0.01"/>
-    </geometry>
-  </collision>
-  </link>
-  <joint name="center_wheel_joint" type="fixed">
-    <origin xyz="-0.0035 0 -0.001" rpy="0 0 0"/>
-    <parent link="center_wheel"/>
-    <child link="center_hubcap"/>
-  </joint>
+      <inertia ixx="0.012411765597" ixy="-0.000711733678" ixz="0.00050272983" iyy="0.015218160428" iyz="-0.000004273467" izz="0.011763977943"/>
+    </inertial>
+    <visual name="base_visual">
+      <origin xyz="0 0 0" rpy="0 0 0"/>
+      <geometry name="pioneer_geom">
+        <mesh filename="package://p2os_urdf/meshes/p3dx_meshes/center_wheel.stl"/>
+      </geometry>
+      <material name="WheelBlack">
+        <color rgba="0.117 0.117 0.117 1"/>
+      </material>
+    </visual>
+    <collision>
+      <origin xyz="0 0 0" rpy="${-PI/2.0} 0 0"/>
+      <geometry>
+        <!--<mesh filename="package://p2os_urdf/meshes/p3dx_meshes/center_wheel.stl"/>-->
+        <cylinder radius="0.0375" length="0.01"/>
+      </geometry>
+    </collision>
+  </link>
   <gazebo reference="center_wheel">
     <material value="Gazebo/Black"/>
@@ -255,7 +262,13 @@
     <elem key="kd"  value="1.0" />
   </gazebo>
-  <xacro:P3DX_WHEEL suffix="left" parent="base_link" reflect="1"/>
-  <xacro:P3DX_WHEEL suffix="right" parent="base_link" reflect="-1"/>
-  <!-- Front + Back Sonar -->
+  <joint name="center_wheel_joint" type="fixed">
+    <origin xyz="-0.0035 0 -0.001" rpy="0 0 0"/>
+    <parent link="center_wheel"/>
+    <child link="center_hubcap"/>
+  </joint>
+  <!-- Wheels -->
+  <xacro:WHEEL name="left" parent="base_link" reflect="1"/>
+  <xacro:WHEEL name="right" parent="base_link" reflect="-1"/>
+  <!-- Sonars -->
   <link name="front_sonar">
     <inertial>
@@ -285,7 +298,7 @@
   </gazebo>
   <joint name="base_front_joint" type="fixed">
-    <origin xyz="-0.198 0 0.208" rpy="0 0 0"/>
     <parent link="base_link"/>
     <child link="front_sonar"/>
+    <origin xyz="-0.198 0 0.208" rpy="0 0 0"/>
   </joint>
   <link name="back_sonar">
@@ -330,4 +343,5 @@
       <interface:position name="position_iface_0"/>
     </controller:differential_position2d>
+    <!--
     <controller:gazebo_ros_p3d name="p3d_base_controller" plugin="libgazebo_ros_p3d.so">
       <alwaysOn>true</alwaysOn>
@@ -337,11 +351,13 @@
       <gaussianNoise>0.01</gaussianNoise>
       <frameName>map</frameName>
-      <xyzOffsets>0 0 0</xyzOffsets> <!-- initialize odometry for fake localization-->
+      <xyzOffsets>0 0 0</xyzOffsets>
       <rpyOffsets>0 0 0</rpyOffsets>
       <interface:position name="p3d_base_position"/>
     </controller:gazebo_ros_p3d>
+    -->
     <!-- this publishes empty joint_states due to no transmission, but
          triggering robot_state_puublisher to publish tf between fixed joints in erratic,
          (e.g. base_laser_link for the base_scan frame) -->
+    <!--
     <controller:gazebo_ros_controller_manager name="gazebo_ros_controller_manager" plugin="libgazebo_ros_controller_manager.so">
       <alwaysOn>true</alwaysOn>
@@ -349,4 +365,5 @@
       <interface:audio name="gazebo_ros_controller_manager_dummy_iface" />
     </controller:gazebo_ros_controller_manager>
+    -->
   </gazebo>
 </robot>

File: packages/my_gazebo_worlds/worlds/empty.world.xacro (robot description, xacro)
@@ -42,5 +42,8 @@
     </model:renderable>
   </xacro:macro>
-  <!-- Macro to create point lights distributed around the world -->
+  <!--
+    Macro to create point lights distributed around the world.  This is just an easy way to get
+    light everwhere.  If we could spawn lights we might choose to spawn lights as needed instead.
+  -->
   <xacro:macro name="LIGHTS_MACRO">
     <xacro:LIGHT_MACRO n="1" x="0"                y="0"               z="${LIGHT_HEIGHT}" />
@@ -53,24 +56,40 @@
   <!-- END XACRO DEFINITIONS        -->
   <!-- ============================ -->
+  <!-- General -->
   <thread>4</thread>
   <verbosity>5</verbosity>
+  <!-- Physics -->
   <physics:ode>
+    <!-- Gravity (m/s^2) -->
+    <gravity>0 0 -9.8</gravity>
+    <!-- Physics engine step duration (s) -->
     <stepTime>0.001</stepTime>
-    <gravity>0 0 -9.8</gravity>
-    <cfm>1e-10</cfm>
-    <erp>0.2</erp>
+    <!-- Physics engine step parameters -->
     <stepType>quick</stepType>
     <stepIters>10</stepIters>
     <stepW>1.3</stepW>
-    <contactMaxCorrectingVel>100.0</contactMaxCorrectingVel>
-    <contactSurfaceLayer>0.001</contactSurfaceLayer>
+    <!-- Constraint force mixing (stiffness) -->
+    <cfm>1e-10</cfm>
+    <!-- Error reduction parameter (damping) -->
+    <erp>0.2</erp>
+    <!-- Maximum velocity that a contact can generate (m/s) -->
+    <contactMaxCorrectingVel>10.0</contactMaxCorrectingVel>
+    <!-- Depth to which contacts may sink (m) -->
+    <contactSurfaceLayer>0.005</contactSurfaceLayer>
   </physics:ode>
+  <!-- Geographical origin -->
   <geo:origin>
-    <lat>43.24355</lat><lon>-5.776711</lon>
+    <lat>43.24355</lat>
+    <lon>-5.776711</lon>
   </geo:origin>
+  <!-- GUI -->
   <rendering:gui>
+    <!-- GUI type, for now only fltk exists -->
     <type>fltk</type>
+    <!-- GUI window size -->
     <size>480 320</size>
+    <!-- GUI window position -->
     <pos>0 0</pos>
+    <!-- GUI frames loaded initially -->
     <frames>
       <row height="100%">
@@ -82,6 +101,7 @@
     </frames>
   </rendering:gui>
+  <!-- Rendering settings -->
   <rendering:ogre>
-    <ambient>0.6 0.6 0.6 0.6</ambient>
+    <ambient>0.4 0.4 0.4 0.4</ambient>
     <sky>
       <material>Gazebo/CloudySky</material>
@@ -92,4 +112,5 @@
     <shadows>false</shadows>
   </rendering:ogre>
+  <!-- Ground -->
   <model:physical name="ground">
     <xyz>0 0 0</xyz>
@@ -106,9 +127,10 @@
         <size>${GROUND_PLANE_SIZE} ${GROUND_PLANE_SIZE}</size>
         <segments>10 10</segments>
-        <uvTile>200 400</uvTile>
+        <uvTile>${GROUND_PLANE_SIZE*2} ${GROUND_PLANE_SIZE*4}</uvTile>
         <material>Gazebo/GrayGrid</material>
       </geom:plane>
     </body:plane>
   </model:physical>
+  <!-- Lights -->
   <xacro:LIGHTS_MACRO/>
 </gazebo:world>
