Commit message: Updating launch files, robot descriptions, and empty world.

File: packages/my_gazebo_worlds/models/pioneer2dx.model.xacro (robot description, xacro)
@@ -13,9 +13,11 @@
   <!-- BEGIN XACRO DEFINITIONS      -->
   <!-- ============================ -->
+  <!-- Height to elevate all parts -->
+  <xacro:property name="HEIGHT" value="0.15"/>
   <!-- Macro to create a wheel -->
   <xacro:macro name="WHEEL" params="name parent reflect">
     <!-- Wheel body -->
     <body:cylinder name="${name}_wheel">
-      <xyz>0.1 ${-reflect*0.17} -0.0725</xyz>
+      <xyz>0.1 ${-reflect*0.17} ${-0.0725 + HEIGHT}</xyz>
       <rpy>0 90 90</rpy>
       <geom:cylinder name="${name}_wheel_geom">
@@ -44,5 +46,5 @@
     </body:cylinder>
     <!-- Join wheel and base_link -->
-    <joint:hinge name="${name}_wheel_hinge">
+    <joint:hinge name="${name}_wheel_joint">
       <body1>${name}_wheel</body1>
       <body2>base_link</body2>
@@ -62,5 +64,5 @@
   <!-- Base link -->
   <body:box name="base_link">
-    <xyz>0.0 0.0 0.0</xyz>
+    <xyz>0.0 0.0 ${0.0 + HEIGHT}</xyz>
     <rpy>0.0 0.0 0.0</rpy>
     <geom:box name="base_link_geom">
@@ -77,5 +79,5 @@
       </visual>
       <visual>
-        <xyz>0.015 0 0.09</xyz>
+        <xyz>0.015 0 0.0975</xyz>
         <rpy>0 0 0</rpy>
         <mesh>Pioneer2at/chassis_top.mesh</mesh>
@@ -100,5 +102,5 @@
   <!-- Castor -->
   <body:sphere name="castor">
-    <xyz>-0.200 0 -0.108</xyz>
+    <xyz>-0.200 0 ${-0.108 + HEIGHT}</xyz>
     <rpy>0 0 0</rpy>
     <geom:sphere name="castor_geom">
@@ -125,6 +127,7 @@
   <!-- Controller -->
   <controller:differential_position2d name="controller1">
-    <leftJoint>left_wheel_hinge</leftJoint>
-    <rightJoint>right_wheel_hinge</rightJoint>
+    <update>100</update>
+    <leftJoint>left_wheel_joint</leftJoint>
+    <rightJoint>right_wheel_joint</rightJoint>
     <wheelSeparation>0.34</wheelSeparation>
     <wheelDiameter>0.15</wheelDiameter>

File: packages/my_gazebo_worlds/models/pioneer3dx.urdf.xacro (robot description, xacro)
@@ -73,5 +73,5 @@
     </gazebo>
     <!-- Join wheel and hubcap -->
-    <joint name="base_${name}_hubcap_joint" type="fixed">
+    <joint name="${name}_hubcap_joint" type="fixed">
       <parent link="${name}_wheel"/>
       <child link="${name}_hubcap"/>
@@ -79,5 +79,5 @@
     </joint>
     <!-- Join wheel and base_link -->
-    <joint name="base_${name}_wheel_joint" type="continuous">
+    <joint name="${name}_wheel_joint" type="continuous">
       <parent link="base_link"/>
       <child link="${name}_wheel"/>
@@ -89,6 +89,6 @@
     <!--
     <transmission name="${parent}_${name}_wheel_trans" type="pr2_mechanism_model/SimpleTransmission">
-      <actuator name="base_${name}_wheel_motor"/>
-      <joint name="base_${name}_wheel_joint"/>
+      <actuator name="${name}_wheel_motor"/>
+      <joint name="${name}_wheel_joint"/>
       <mechanicalReduction>${reflect * 624/35 * 80/19}</mechanicalReduction>
     </transmission>
@@ -154,5 +154,5 @@
   </gazebo>
   <!-- Join top_plate and base_link -->
-  <joint name="base_top_joint" type="fixed">
+  <joint name="top_joint" type="fixed">
     <parent link="base_link"/>
     <child link="top_plate"/>
@@ -184,5 +184,5 @@
   </gazebo>
   <!-- Join swivel and base_link -->
-  <joint name="base_swivel_joint" type="continuous">
+  <joint name="swivel_joint" type="continuous">
     <parent link="base_link"/>
     <child link="swivel"/>
@@ -287,5 +287,5 @@
   </gazebo>
   <!-- Join front_sonar and base_link -->
-  <joint name="base_front_joint" type="fixed">
+  <joint name="front_joint" type="fixed">
     <parent link="base_link"/>
     <child link="front_sonar"/>
@@ -317,5 +317,5 @@
   </gazebo>
   <!-- Join back_sonar and base_link -->
-  <joint name="base_back_joint" type="fixed">
+  <joint name="back_joint" type="fixed">
     <parent link="base_link"/>
     <child link="back_sonar"/>
@@ -326,6 +326,6 @@
     <controller:differential_position2d name="controller1">
       <update>100</update>
-      <leftJoint>base_right_wheel_joint</leftJoint>
-      <rightJoint>base_left_wheel_joint</rightJoint>
+      <leftJoint>left_wheel_joint</leftJoint>
+      <rightJoint>right_wheel_joint</rightJoint>
       <wheelSeparation>0.39</wheelSeparation>
       <wheelDiameter>0.15</wheelDiameter>
@@ -338,5 +338,5 @@
       <updateRate>100.0</updateRate>
       <bodyName>base_link</bodyName>
-      <topicName>base_pose_ground_truth</topicName>
+      <topicName>pose_ground_truth</topicName>
       <gaussianNoise>0.01</gaussianNoise>
       <frameName>map</frameName>

File: packages/my_gazebo_worlds/worlds/empty.world.xacro (robot description, xacro)
@@ -127,5 +127,5 @@
         <size>${GROUND_PLANE_SIZE} ${GROUND_PLANE_SIZE}</size>
         <segments>10 10</segments>
-        <uvTile>${GROUND_PLANE_SIZE*2} ${GROUND_PLANE_SIZE*4}</uvTile>
+        <uvTile>${GROUND_PLANE_SIZE} ${GROUND_PLANE_SIZE}</uvTile>
         <material>Gazebo/GrayGrid</material>
       </geom:plane>

Commit message: Updates.

File: packages/my_gazebo_worlds/models/pioneer2dx.model.xacro (robot description, xacro)
@@ -13,5 +13,5 @@
   <!-- BEGIN XACRO DEFINITIONS      -->
   <!-- ============================ -->
-  <!-- Height to elevate all parts -->
+  <!-- Height to elevate all parts to avoid collision with the ground-->
   <xacro:property name="HEIGHT" value="0.15"/>
   <!-- Macro to create a wheel -->
@@ -115,5 +115,5 @@
   </body:sphere>
   <!-- Join castor and base_link -->
-  <joint:ball name="ball_joint">
+  <joint:ball name="castor_joint">
     <body1>castor</body1>
     <body2>base_link</body2>

File: packages/my_gazebo_worlds/models/pioneer3dx.urdf.xacro (robot description, xacro)
@@ -221,5 +221,5 @@
   </gazebo>
   <!-- Join center_wheel and swivel -->
-  <joint name="swivel_hubcap_joint" type="continuous">
+  <joint name="center_wheel_joint" type="continuous">
     <parent link="swivel"/>
     <child link="center_wheel"/>
@@ -254,73 +254,73 @@
   </gazebo>
   <!-- Join center_wheel and center_hubcap -->
-  <joint name="center_wheel_joint" type="fixed">
+  <joint name="center_hubcap_joint" type="fixed">
     <parent link="center_wheel"/>
     <child link="center_hubcap"/>
     <origin xyz="-0.0035 0 -0.001" rpy="0 0 0"/>
   </joint>
+  <!-- Front sonars -->
+  <link name="front_sonar">
+    <inertial>
+      <mass value="0.0001"/>
+      <origin xyz="0 0 0"/>
+      <inertia ixx="1" ixy="0" ixz="0" iyy="1" iyz="0" izz="1"/>
+    </inertial>
+    <visual>
+      <origin xyz="0 0 0" rpy="0 0 0"/>
+      <geometry>
+        <mesh filename="package://p2os_urdf/meshes/p3dx_meshes/front_sonar.stl"/>
+      </geometry>
+      <material name="SonarYellow"/>
+    </visual>
+    <collision>
+      <origin xyz="0 0 0" rpy="0 0 0"/>
+      <geometry>
+        <box size="0 0 0"/>
+      </geometry>
+    </collision>
+  </link>
+  <gazebo reference="front_sonar">
+    <material value="Gazebo/Yellow"/>
+  </gazebo>
+  <!-- Join front_sonar and base_link -->
+  <joint name="front_sonar_joint" type="fixed">
+    <parent link="base_link"/>
+    <child link="front_sonar"/>
+    <origin xyz="-0.198 0 0.208" rpy="0 0 0"/>
+  </joint>
+  <!-- Back sonars -->
+  <link name="back_sonar">
+    <inertial>
+      <mass value="0.0001"/>
+      <origin xyz="0 0 0"/>
+      <inertia ixx="1" ixy="0" ixz="0" iyy="1" iyz="0" izz="1"/>
+    </inertial>
+    <visual>
+      <origin xyz="0 0 0" rpy="0 0 0"/>
+      <geometry>
+        <mesh filename="package://p2os_urdf/meshes/p3dx_meshes/back_sonar.stl"/>
+      </geometry>
+      <material name="SonarYellow"/>
+    </visual>
+    <collision>
+      <origin xyz="0 0 0" rpy="0 0 0"/>
+      <geometry>
+        <box size="0 0 0"/>
+      </geometry>
+    </collision>
+  </link>
+  <gazebo reference="back_sonar">
+    <material value="Gazebo/Yellow"/>
+  </gazebo>
+  <!-- Join back_sonar and base_link -->
+  <joint name="back_sonar_joint" type="fixed">
+    <parent link="base_link"/>
+    <child link="back_sonar"/>
+    <origin xyz="0.109 0 0.209" rpy="0 0 0"/>
+  </joint>
   <!-- Wheels -->
   <xacro:WHEEL name="left" parent="base_link" reflect="1"/>
   <xacro:WHEEL name="right" parent="base_link" reflect="-1"/>
-  <!-- Front sonars -->
-  <link name="front_sonar">
-    <inertial>
-      <mass value="0.0001"/>
-      <origin xyz="0 0 0"/>
-      <inertia ixx="1" ixy="0" ixz="0" iyy="1" iyz="0" izz="1"/>
-    </inertial>
-    <visual>
-      <origin xyz="0 0 0" rpy="0 0 0"/>
-      <geometry>
-        <mesh filename="package://p2os_urdf/meshes/p3dx_meshes/front_sonar.stl"/>
-      </geometry>
-      <material name="SonarYellow"/>
-    </visual>
-    <collision>
-      <origin xyz="0 0 0" rpy="0 0 0"/>
-      <geometry>
-        <box size="0 0 0"/>
-      </geometry>
-    </collision>
-  </link>
-  <gazebo reference="front_sonar">
-    <material value="Gazebo/Yellow"/>
-  </gazebo>
-  <!-- Join front_sonar and base_link -->
-  <joint name="front_joint" type="fixed">
-    <parent link="base_link"/>
-    <child link="front_sonar"/>
-    <origin xyz="-0.198 0 0.208" rpy="0 0 0"/>
-  </joint>
-  <!-- Back sonars -->
-  <link name="back_sonar">
-    <inertial>
-      <mass value="0.0001"/>
-      <origin xyz="0 0 0"/>
-      <inertia ixx="1" ixy="0" ixz="0" iyy="1" iyz="0" izz="1"/>
-    </inertial>
-    <visual>
-      <origin xyz="0 0 0" rpy="0 0 0"/>
-      <geometry>
-        <mesh filename="package://p2os_urdf/meshes/p3dx_meshes/back_sonar.stl"/>
-      </geometry>
-      <material name="SonarYellow"/>
-    </visual>
-    <collision>
-      <origin xyz="0 0 0" rpy="0 0 0"/>
-      <geometry>
-        <box size="0 0 0"/>
-      </geometry>
-    </collision>
-  </link>
-  <gazebo reference="back_sonar">
-    <material value="Gazebo/Yellow"/>
-  </gazebo>
-  <!-- Join back_sonar and base_link -->
-  <joint name="back_joint" type="fixed">
-    <parent link="base_link"/>
-    <child link="back_sonar"/>
-    <origin xyz="0.109 0 0.209" rpy="0 0 0"/>
-  </joint>
-  <!-- Connect controllers -->
+  <!-- Controllers -->
   <gazebo>
     <controller:differential_position2d name="controller1">
