Commit message: New structure -- temp commit.

File: my_gazebo_worlds/worlds/empty.world.xacro (robot description, xacro)
@@ -23,19 +23,35 @@
   <!-- ============================ -->
   <!-- Ground plane size in metres (both x and y) -->
-  <xacro:property name="GROUND_PLANE_SIZE"  value="100" />
+  <xacro:property name="GROUND_PLANE_SIZE"  value="100.0" />
   <!-- Range and height for each light -->
   <xacro:property name="LIGHT_RANGE"        value="${GROUND_PLANE_SIZE/4}" />
-  <xacro:property name="LIGHT_HEIGHT"       value="10" />
+  <xacro:property name="LIGHT_HEIGHT"       value="10.0" />
   <!-- Macro to create one point light at given position -->
   <xacro:macro name="LIGHT_MACRO" params="n x y z">
     <model:renderable name="light_${n}">
+      <!-- Affected by gravity -->
+      <enableGravity>false</enableGravity>
+      <!-- Light pose (only needed for point or spot) -->
       <xyz>${x} ${y} ${z}</xyz>
-      <rpy>0.0 0.0 0</rpy>
-      <enableGravity>false</enableGravity>
+      <rpy>0.0 0.0 0.0</rpy>
+      <!-- Light parameters -->
       <light>
+        <!-- Light type (point, directional, or spot) -->
         <type>point</type>
+        <!-- Light direction vector (only for directional or spot) -->
+        <direction>0.0 0.0 -1.0</direction>
+        <!-- Spotlight parameters (only for spot) -->
+        <innerAngle>10.0</innerAngle>
+        <outerAngle>20.0</outerAngle>
+        <falloff>1.0</falloff>
+        <!-- Cast shadows -->
+        <castShadows>true</castShadows>
+        <!-- Diffuse colour (matte surfaces) in RGB ([0,1]) -->
         <diffuseColor>0.8 0.8 0.8</diffuseColor>
-        <specularColor>.1 .1 .1</specularColor>
-        <attenuation>0.2 0.1 0</attenuation>
+        <!-- Specular colour (glossy surfaces) in RGB ([0,1]) -->
+        <specularColor>0.1 0.1 0.1</specularColor>
+        <!-- Attenuation over range (constant, linear, quadratic) -->
+        <attenuation>0.2 0.1 0.0</attenuation>
+        <!-- Light range (m) -->
         <range>${LIGHT_RANGE}</range>
       </light>
@@ -62,10 +78,10 @@
   <physics:ode>
     <!-- Gravity (m/s^2) -->
-    <gravity>0 0 -9.8</gravity>
+    <gravity>0.0 0.0 -9.8</gravity>
     <!-- Physics engine step duration (s) -->
     <stepTime>0.001</stepTime>
     <!-- Physics engine step parameters -->
     <stepType>quick</stepType>
-    <stepIters>10</stepIters>
+    <stepIters>10.0</stepIters>
     <stepW>1.3</stepW>
     <!-- Constraint force mixing (stiffness) -->
@@ -103,4 +119,5 @@
   <!-- Rendering settings -->
   <rendering:ogre>
+    <!-- Ambient light -->
     <ambient>0.4 0.4 0.4 0.4</ambient>
     <sky>
@@ -114,6 +131,6 @@
   <!-- Ground -->
   <model:physical name="ground">
-    <xyz>0 0 0</xyz>
-    <rpy>0 0 0</rpy>
+    <xyz>0.0 0.0 0.0</xyz>
+    <rpy>0.0 0.0 0.0</rpy>
     <static>true</static>
     <body:plane name="ground_body">
@@ -124,5 +141,5 @@
         <kp>1000000000.0</kp>
         <kd>1.0</kd>
-        <normal>0 0 1</normal>
+        <normal>0.0 0.0 1.0</normal>
         <size>${GROUND_PLANE_SIZE} ${GROUND_PLANE_SIZE}</size>
         <segments>10 10</segments>
